File: resources/kicad/Acceleration Logger/Acceleration Logger.kicad_sch (KiCad schematic)
At the start: 12 parts, among them J1 Screw_Terminal_01x02, J2 USB_B_Micro, Q1 2N3904, U1 ESP8266-01s, U2 MPU6050, U3 MCP1700x-330xxTO

Commit message: Many updates
Parts:
- added R3: 1K, Resistor_SMD:R_0805_2012Metric_Pad1.20x1.40mm_HandSolder, symbol Device:R_Small_US
Connections:
- net +3V3: now also R3.1
- net SDA: now reaches DISP1.4 (SDA), U1.5 (GPIO0), U2.4 (SDA)
- net at D1.2 (A), R2.1: now also U1.2 (U0TXD/GPIO1), R3.2; no longer U1.7 (GPIO3/U0RXD)
- net at U2.8 (INT): now also U1.7 (GPIO3/U0RXD); no longer U1.2 (U0TXD/GPIO1)
Changed lines of the file:
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@@
 		(title "Acceleration Logger")
 		(date "2025-03-06")
-		(rev "0.0.1")
+		(rev "0.0.2")
 	)
 	(junction
@@
 	)
 	(junction
-		(at 121.158 90.932)
+		(at 121.158 76.454)
 		(diameter 0)
 		(color 0 0 0 0)
@@
 	(wire
 		(pts
+			(xy 138.938 106.68) (xy 138.938 114.554)
+		)
+		(stroke
+			(width 0)
+			(type default)
+		)
+	)
+	(wire
+		(pts
 			(xy 163.576 89.662) (xy 163.576 96.52)
 		)
@@
 	(wire
 		(pts
-			(xy 121.158 114.554) (xy 121.158 90.932)
-		)
-		(stroke
-			(width 0)
-			(type default)
-		)
-	)
-	(wire
-		(pts
 			(xy 134.366 122.428) (xy 137.922 122.428)
 		)
@@
 	(wire
 		(pts
-			(xy 119.888 114.554) (xy 121.158 114.554)
+			(xy 121.158 70.612) (xy 121.158 76.454)
 		)
 		(stroke
@@
 	(wire
 		(pts
-			(xy 78.74 137.922) (xy 78.74 122.174)
-		)
-		(stroke
-			(width 0)
-			(type default)
-		)
-	)
-	(wire
-		(pts
 			(xy 134.366 117.094) (xy 134.366 122.428)
 		)
@@
 	(wire
 		(pts
-			(xy 183.388 137.922) (xy 78.74 137.922)
-		)
-		(stroke
-			(width 0)
-			(type default)
-		)
-	)
-	(wire
-		(pts
 			(xy 127 90.678) (xy 127 94.234)
 		)
@@
 	(wire
 		(pts
-			(xy 183.388 113.538) (xy 183.388 137.922)
-		)
-		(stroke
-			(width 0)
-			(type default)
-		)
-	)
-	(wire
-		(pts
 			(xy 84.328 59.182) (xy 88.646 59.182)
 		)
@@
 	(wire
 		(pts
-			(xy 141.224 113.538) (xy 183.388 113.538)
-		)
-		(stroke
-			(width 0)
-			(type default)
-		)
-	)
-	(wire
-		(pts
-			(xy 78.74 122.174) (xy 81.788 122.174)
-		)
-		(stroke
-			(width 0)
-			(type default)
-		)
-	)
-	(wire
-		(pts
 			(xy 97.282 90.932) (xy 97.282 94.742)
 		)
@@
 	(wire
 		(pts
-			(xy 141.224 106.68) (xy 141.224 113.538)
+			(xy 75.946 122.174) (xy 75.946 76.454)
+		)
+		(stroke
+			(width 0)
+			(type default)
+		)
+	)
+	(wire
+		(pts
+			(xy 81.788 122.174) (xy 75.946 122.174)
 		)
 		(stroke
@@
 	(wire
 		(pts
+			(xy 75.946 76.454) (xy 121.158 76.454)
+		)
+		(stroke
+			(width 0)
+			(type default)
+		)
+	)
+	(wire
+		(pts
 			(xy 64.262 58.42) (xy 71.628 58.42)
 		)
@@
 	(wire
 		(pts
+			(xy 141.224 106.68) (xy 138.938 106.68)
+		)
+		(stroke
+			(width 0)
+			(type default)
+		)
+	)
+	(wire
+		(pts
+			(xy 121.158 60.96) (xy 121.158 65.532)
+		)
+		(stroke
+			(width 0)
+			(type default)
+		)
+	)
+	(wire
+		(pts
 			(xy 172.212 84.074) (xy 172.212 80.01)
 		)
@@
 		(pts
 			(xy 119.888 119.634) (xy 131.318 119.634)
+		)
+		(stroke
+			(width 0)
+			(type default)
+		)
+	)
+	(wire
+		(pts
+			(xy 138.938 114.554) (xy 119.888 114.554)
 		)
 		(stroke
@@
 	(label "+5V"
 		(at 74.168 59.182 0)
+		(effects
+			(font
+				(size 1.27 1.27)
+			)
+			(justify left bottom)
+		)
+	)
+	(label "SCL"
+		(at 120.396 119.888 0)
+		(effects
+			(font
+				(size 1.27 1.27)
+			)
+			(justify left bottom)
+		)
+	)
+	(label "SDA"
+		(at 120.396 117.094 0)
 		(effects
 			(font
@@
 	)
 	(symbol
+		(lib_id "power:+3V3")
+		(at 121.158 60.96 0)
+		(unit 1)
+		(exclude_from_sim no)
+		(in_bom yes)
+		(on_board yes)
+		(dnp no)
+		(fields_autoplaced yes)
+		(property "Reference" "#PWR015"
+			(at 121.158 64.77 0)
+			(effects
+				(font
+					(size 1.27 1.27)
+				)
+				(hide yes)
+			)
+		)
+		(property "Value" "+3V3"
+			(at 121.158 56.642 0)
+			(effects
+				(font
+					(size 1.27 1.27)
+				)
+			)
+		)
+		(property "Footprint" ""
+			(at 121.158 60.96 0)
+			(effects
+				(font
+					(size 1.27 1.27)
+				)
+				(hide yes)
+			)
+		)
+		(property "Datasheet" ""
+			(at 121.158 60.96 0)
+			(effects
+				(font
+					(size 1.27 1.27)
+				)
+				(hide yes)
+			)
+		)
+		(property "Description" "Power symbol creates a global label with name \"+3V3\""
+			(at 121.158 60.96 0)
+			(effects
+				(font
+					(size 1.27 1.27)
+				)
+				(hide yes)
+			)
+		)
+		(pin "1"
+		)
+		(instances
+			(project "Acceleration Logger"
+				(path "/9ffc3f79-5742-486a-81da-0f55a501c912"
+					(reference "#PWR015")
+					(unit 1)
+				)
+			)
+		)
+	)
+	(symbol
 		(lib_id "Device:LED_Small")
 		(at 106.68 90.932 0)
@@
 					(unit 1)
 				)
+			)
+		)
+	)
+	(symbol
+		(lib_id "Device:R_Small_US")
+		(at 121.158 68.072 0)
+		(unit 1)
+		(exclude_from_sim no)
+		(in_bom yes)
+		(on_board yes)
+		(dnp no)
+		(fields_autoplaced yes)
+		(property "Reference" "R3"
+			(at 122.936 66.8019 0)
+			(effects
+				(font
+					(size 1.27 1.27)
+				)
+				(justify left)
+			)
+		)
+		(property "Value" "1K"
+			(at 122.936 69.3419 0)
+			(effects
+				(font
+					(size 1.27 1.27)
+				)
+				(justify left)
+			)
+		)
+		(property "Footprint" "Resistor_SMD:R_0805_2012Metric_Pad1.20x1.40mm_HandSolder"
+			(at 121.158 68.072 0)
+			(effects
+				(font
+					(size 1.27 1.27)
+				)
+				(hide yes)
+			)
+		)
+		(property "Datasheet" "~"
+			(at 121.158 68.072 0)
+			(effects
+				(font
+					(size 1.27 1.27)
+				)
+				(hide yes)
+			)
+		)
+		(property "Description" "Resistor, small US symbol"
+			(at 121.158 68.072 0)
+			(effects
+				(font
+					(size 1.27 1.27)
+				)
+				(hide yes)
+			)
+		)
+		(pin "2"
+		)
+		(pin "1"
+		)
+		(instances
+			(project "Acceleration Logger"
+				(path "/9ffc3f79-5742-486a-81da-0f55a501c912"
+					(reference "R3")
+					(unit 1)
+				)

Commit message: Board updates
Parts:
- J1: value Screw_Terminal_01x02 -> Vehicle Brakes
- Q1: value 2N3904 -> IRLML6344; symbol Davids_Symbols:NPN_Transistor_with_correct_pinout_for_SOT-23 -> Transistor_FET:IRLML6244
- R2: value 1K -> 330
- R3: value 1K -> 10K
Connections:
- net +3V3: no longer J1.1 (Pin_1)
- net Earth: now also J1.2 (Pin_2)
- net at Q1.3 (D): now also J1.1 (Pin_1); no longer J1.2 (Pin_2)
Other:
- note added: "Brake +12v"
- note added: "Brake -"
- title: Acceleration Logger -> Acceleration Logger and indicator
- moved on the sheet: J1
Changed lines of the file:
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@@
 	(paper "A4")
 	(title_block
-		(title "Acceleration Logger")
-		(date "2025-03-06")
-		(rev "0.0.2")
+		(title "Acceleration Logger and indicator")
+		(date "2025-04-07")
+		(rev "0.1.0")
 	)
 	(junction
@@
 	(wire
 		(pts
-			(xy 172.212 86.614) (xy 178.308 86.614)
-		)
-		(stroke
-			(width 0)
-			(type default)
-		)
-	)
-	(wire
-		(pts
 			(xy 84.328 66.548) (xy 84.328 69.088)
 		)
@@
 	(wire
 		(pts
+			(xy 188.468 96.52) (xy 186.69 96.52)
+		)
+		(stroke
+			(width 0)
+			(type default)
+		)
+	)
+	(wire
+		(pts
 			(xy 163.576 76.454) (xy 163.576 84.582)
 		)
@@
 	(wire
 		(pts
+			(xy 186.69 96.52) (xy 186.69 104.14)
+		)
+		(stroke
+			(width 0)
+			(type default)
+		)
+	)
+	(wire
+		(pts
 			(xy 134.366 122.428) (xy 137.922 122.428)
 		)
@@
 	(wire
 		(pts
-			(xy 172.212 91.44) (xy 172.212 86.614)
+			(xy 186.69 93.98) (xy 186.69 89.662)
 		)
 		(stroke
@@
 	(wire
 		(pts
-			(xy 178.308 84.074) (xy 172.212 84.074)
+			(xy 188.468 93.98) (xy 186.69 93.98)
+		)
+		(stroke
+			(width 0)
+			(type default)
+		)
+	)
+	(wire
+		(pts
+			(xy 186.69 89.662) (xy 172.212 89.662)
 		)
 		(stroke
@@
 	(wire
 		(pts
+			(xy 172.212 89.662) (xy 172.212 91.44)
+		)
+		(stroke
+			(width 0)
+			(type default)
+		)
+	)
+	(wire
+		(pts
 			(xy 131.318 119.634) (xy 131.318 124.968)
 		)
@@
 	(wire
 		(pts
-			(xy 172.212 84.074) (xy 172.212 80.01)
-		)
-		(stroke
-			(width 0)
-			(type default)
-		)
-	)
-	(wire
-		(pts
 			(xy 119.888 119.634) (xy 131.318 119.634)
 		)
@@
 			(width 0)
 			(type default)
+		)
+	)
+	(text "Brake -"
+		(exclude_from_sim no)
+		(at 199.39 97.028 0)
+		(effects
+			(font
+				(size 1.27 1.27)
+			)
+		)
+	)
+	(text "Brake +12v"
+		(exclude_from_sim no)
+		(at 200.914 93.98 0)
+		(effects
+			(font
+				(size 1.27 1.27)
+			)
 		)
 	)
@@
 	(symbol
 		(lib_id "Connector:Screw_Terminal_01x02")
-		(at 183.388 84.074 0)
-		(unit 1)
-		(exclude_from_sim no)
-		(in_bom yes)
-		(on_board yes)
-		(dnp no)
-		(fields_autoplaced yes)
+		(at 193.548 93.98 0)
+		(unit 1)
+		(exclude_from_sim no)
+		(in_bom yes)
+		(on_board yes)
+		(dnp no)
 		(property "Reference" "J1"
-			(at 185.42 84.0739 0)
+			(at 192.024 90.932 0)
 			(effects
 				(font
@@
 			)
 		)
-		(property "Value" "Screw_Terminal_01x02"
-			(at 185.42 86.6139 0)
+		(property "Value" "Vehicle Brakes"
+			(at 188.214 100.33 0)
 			(effects
 				(font
@@
 		)
 		(property "Footprint" "Davids_Footprints:KF350 2 Pin Terminal Block"
-			(at 183.388 84.074 0)
+			(at 193.548 93.98 0)
 			(effects
 				(font
@@
 		)
 		(property "Datasheet" "~"
-			(at 183.388 84.074 0)
+			(at 193.548 93.98 0)
 			(effects
 				(font
@@
 		)
 		(property "Description" "Generic screw terminal, single row, 01x02, script generated (kicad-library-utils/schlib/autogen/connector/)"
-			(at 183.388 84.074 0)
+			(at 193.548 93.98 0)
 			(effects
 				(font
@@
 		(fields_autoplaced yes)
 		(property "Reference" "R3"
-			(at 122.936 66.8019 0)
+			(at 123.19 66.8019 0)
 			(effects
 				(font
@@
 			)
 		)
-		(property "Value" "1K"
-			(at 122.936 69.3419 0)
+		(property "Value" "10K"
+			(at 123.19 69.3419 0)
 			(effects
 				(font
@@
 	)
 	(symbol
-		(lib_id "power:+3V3")
-		(at 172.212 80.01 0)
-		(unit 1)
-		(exclude_from_sim no)
-		(in_bom yes)
-		(on_board yes)
-		(dnp no)
-		(fields_autoplaced yes)
-		(property "Reference" "#PWR09"
-			(at 172.212 83.82 0)
-			(effects
-				(font
-					(size 1.27 1.27)
-				)
-				(hide yes)
-			)
-		)
-		(property "Value" "+3V3"
-			(at 172.212 75.692 0)
-			(effects
-				(font
-					(size 1.27 1.27)
-				)
-			)
-		)
-		(property "Footprint" ""
-			(at 172.212 80.01 0)
-			(effects
-				(font
-					(size 1.27 1.27)
-				)
-				(hide yes)
-			)
-		)
-		(property "Datasheet" ""
-			(at 172.212 80.01 0)
-			(effects
-				(font
-					(size 1.27 1.27)
-				)
-				(hide yes)
-			)
-		)
-		(property "Description" "Power symbol creates a global label with name \"+3V3\""
-			(at 172.212 80.01 0)
-			(effects
-				(font
-					(size 1.27 1.27)
-				)
-				(hide yes)
-			)
-		)
-		(pin "1"
-		)
-		(instances
-			(project "Acceleration Logger"
-				(path "/9ffc3f79-5742-486a-81da-0f55a501c912"
-					(reference "#PWR09")
-					(unit 1)
-				)
-			)
-		)
-	)
-	(symbol
 		(lib_id "Device:R_Small_US")
 		(at 163.576 87.122 0)
@@
 		(fields_autoplaced yes)
 		(property "Reference" "R2"
-			(at 165.354 85.8519 0)
+			(at 166.37 85.8519 0)
 			(effects
 				(font
@@
 			)
 		)
-		(property "Value" "1K"
-			(at 165.354 88.3919 0)
+		(property "Value" "330"
+			(at 166.37 88.3919 0)
 			(effects
 				(font
@@
 				(path "/9ffc3f79-5742-486a-81da-0f55a501c912"
 					(reference "R2")
+					(unit 1)
+				)
+			)
+		)
+	)
+	(symbol
+		(lib_id "power:Earth")
+		(at 186.69 104.14 0)
+		(unit 1)
+		(exclude_from_sim no)
+		(in_bom yes)
+		(on_board yes)
+		(dnp no)
+		(fields_autoplaced yes)
+		(property "Reference" "#PWR9"
+			(at 186.69 110.49 0)
+			(effects
+				(font
+					(size 1.27 1.27)
+				)
+				(hide yes)
+			)
+		)
+		(property "Value" "Earth"
+			(at 186.69 107.95 0)
+			(effects
+				(font
+					(size 1.27 1.27)
+				)
+				(hide yes)
+			)
+		)
+		(property "Footprint" ""
+			(at 186.69 104.14 0)
+			(effects
+				(font
+					(size 1.27 1.27)
+				)
+				(hide yes)
+			)
+		)
+		(property "Datasheet" "~"
+			(at 186.69 104.14 0)
+			(effects
+				(font
+					(size 1.27 1.27)
+				)
+				(hide yes)
+			)
+		)
+		(property "Description" "Power symbol creates a global label with name \"Earth\""
+			(at 186.69 104.14 0)
+			(effects
+				(font
+					(size 1.27 1.27)
+				)
+				(hide yes)
+			)
+		)
+		(pin "1"
+		)
+		(instances
+			(project "Acceleration Logger"
+				(path "/9ffc3f79-5742-486a-81da-0f55a501c912"
+					(reference "#PWR9")
 					(unit 1)
 				)
@@
 	)
 	(symbol
-		(lib_id "Davids_Symbols:NPN_Transistor_with_correct_pinout_for_SOT-23")
+		(lib_id "Transistor_FET:IRLML6244")
 		(at 169.672 96.52 0)
 		(unit 1)
@@
 			)
 		)
-		(property "Value" "2N3904"
+		(property "Value" "IRLML6344"
 			(at 175.26 97.7899 0)
 			(effects
@@
 		)
 		(property "Footprint" "Package_TO_SOT_SMD:SOT-23"
-			(at 174.752 98.552 0)
+			(at 174.752 98.425 0)
 			(effects
 				(font
@@
 			)
 		)
-		(property "Datasheet" "https://www.onsemi.com/pub/Collateral/MMBTA42LT1-D.PDF"
-			(at 162.814 75.438 0)
+		(property "Datasheet" "https://www.infineon.com/dgdl/Infineon-IRLML6244-DataSheet-v01_01-EN.pdf?fileId=5546d462533600a4015356686fed261f"
+			(at 174.752 100.33 0)
 			(effects
 				(font
@@
 			)
 		)
-		(property "Description" "0.5A Ic, 300V Vce, NPN High Voltage Transistor, SOT-23"
-			(at 203.454 87.884 0)
-			(effects
-				(font
+		(property "Description" "6.3A Id, 20V Vds, 21mOhm Rds, N-Channel StrongIRFET Power MOSFET, SOT-23"
+			(at 169.672 96.52 0)
+			(effects
+				(font

Commit message: Added "set level" feature. Changed LED to T1-3/4 size
Parts:
- D1: footprint LED_SMD:LED_1206_3216Metric -> LED_THT:LED_D5.0mm
Other:
- title: Acceleration Logger and indicator -> Acceleration Logger and Indicator
Changed lines of the file:
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@@
 	(paper "A4")
 	(title_block
-		(title "Acceleration Logger and indicator")
-		(date "2025-04-07")
-		(rev "0.1.0")
+		(title "Acceleration Logger and Indicator")
+		(date "2025-04-18")
+		(rev "0.1.1")
 	)
 	(junction
@@
 			)
 		)
-		(property "Footprint" "LED_SMD:LED_1206_3216Metric"
+		(property "Footprint" "LED_THT:LED_D5.0mm"
 			(at 95.758 90.424 90)
 			(effects
